File: PCB/Stenokey.kicad_pcb (KiCad board)
At the start: 2 copper layers, 219 x 139.5 mm, 51 parts, among them SW1 KEY_R1C1, SW10 KEY_R1C10, SW11 KEY_R2C1, SW12 KEY_R2C2, SW13 KEY_R2C3, SW14 KEY_R2C4, SW15 KEY_R2C5, SW16 KEY_R2C6, SW17 KEY_R2C7, SW18 KEY_R2C8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

Commit message: implement PULL_DOWN internal pico resistor
Other:
- board text added: "Pico"
